File: EEprom_Logger_V1.brd (EAGLE design)
At the start: 64.7 x 48.5 mm, 25 parts, among them IC1 AP2138N-3.3TRG1, IC2 PIC18F13K22SOP, IC3 MIC94090, IC4 MCP1700T-2702E/TT, IC5 24LC16BSN, Q1 Si2333CDS-T1-GE3, Q2 Si2333CDS-T1-GE3, Y1 32kHz

Commit message: Add files via upload
Parts:
- removed Q1, Q2: Si2333CDS-T1-GE3, SparkFun-DiscreteSemi:SOT23-3
- added R4: 1k, SparkFun-Resistors:1206
- added U$2, U$3: LM66100, LM66100:SC70-6
- C4: value 10uF -> 22uF
- moved C4 7.04 mm to (17.0, 10.2), turned to 90 degrees
Connections:
- new net N$3: C4.2, IC1.2, R4.2, U$2.1
- net 3V: now also U$2.6, U$3.6; no longer Q1.2, Q2.2
- net GND: now also U$2.2, U$3.2; no longer Q1.1, Q2.1
- net N$6: now also R4.1, U$2.5, U$3.3; no longer C4.2, IC1.2, Q2.3
- net N$9: now also U$2.3, U$3.1; no longer Q1.3
